Commit message: changed the dimesnions of the cylinder

File: models/TESTCYLINDER/TESTCYLINDER.urdf (robot description, URDF)
Before this commit: robot TESTCYLINDER, 1 links, 0 joints
Links:
- link TESTCYLINDER__link_0: geometry collision cylinder length=0.045716 radius=0.279343; visual cylinder length=0.00457156 radius=0.079343

Commit message: commented the collision properties in testcylinder.urdf

File: models/TESTCYLINDER/TESTCYLINDER.urdf (robot description, URDF)
Before this commit: robot TESTCYLINDER, 1 links, 0 joints
Links:
- link TESTCYLINDER__link_0: geometry visual cylinder length=0.00457156 radius=0.079343

Commit message: modified the testCylinder URDF and scan_process.py

File: models/TESTCYLINDER/TESTCYLINDER.urdf (robot description, URDF)
Before this commit: robot TESTCYLINDER, 1 links, 0 joints
Links:
- removed link TESTCYLINDER__link_0
- added link base_link, mass 0.0151727; collision cylinder length=0.00001 radius=0.001; visual cylinder length=0.01 radius=0.079343
